File: guitar_booster/guitar_booster.kicad_pcb (KiCad board)
At the start: 2 copper layers, 36 x 23.9 mm, 21 parts, among them J1 Conn_01x02_Pin, J2 Conn_01x02_Pin, SW1.1 KBB40-2P2W, SW1.2 KBB40-2P2W, SW2 SW_DPST_x2

Commit message: Add files via upload
Parts:
- added C4: 10мкФ, Capacitor_SMD:C_0603_1608Metric, F.Cu at (119.5, 82.0)
- added C5: 0,1мкФ, Capacitor_SMD:C_0603_1608Metric, F.Cu at (121.4, 82.0)
Routing:
- net +3V: track 41.0 -> 43.5 mm
