File: guitar_booster/guitar_booster.kicad_sch (KiCad schematic)
At the start: 22 parts, among them J1 Conn_01x02_Pin, J2 Conn_01x02_Pin, SW1.1 KBB40-2P2W, SW1.2 KBB40-2P2W, SW2 SW_DPST_x2, SW3 SW_DPST_x2

Commit message: Add files via upload
Parts:
- added C4: 10мкФ, Capacitor_SMD:C_0603_1608Metric, symbol Device:C
- added C5: 0,1мкФ, Capacitor_SMD:C_0603_1608Metric, symbol Device:C
Connections:
- net +3V: now also C4.2, C5.2
- net GND: now also C4.1, C5.1
Other:
- moved on the sheet: BT1, R8, SW2A, SW3B, VD1
